Commit message: Added a third caster wheel to the urdf as a support.

File: robot_urdf.urdf (robot description, URDF)
Before this commit: robot my_robot, 3 links, 2 joints
Links:
- added link caster_wheel; visual sphere radius=0.05
Joints:
- added joint base_caster_joint: type fixed, parent base_link, child caster_wheel, origin xyz=0.15 0 -0.075 rpy=0 0 0
